Commit message: marco: added missing collision to urdf

File: hrc_simulator_descriptions/urdf/elmo_linear_guide.urdf.xacro (robot description, xacro)
@@ -13,4 +13,13 @@
         </material>
       </visual>
+      <collision>
+        <origin xyz="1 0.0 -0.1" rpy="0 0 0" />
+        <geometry>
+          <box size="2.2 0.3 0.2"/>
+        </geometry>
+        <material name="DarkGrey">
+          <color rgba="0.4 0.4 0.4 1.0"/>
+        </material>
+      </collision>
       <inertial>
           <origin xyz="0 0 0" rpy="0 0 0" />

File: hrc_simulator_descriptions/urdf/wheeled_table_dim.urdf.xacro (robot description, xacro)
@@ -12,4 +12,13 @@
       </material>
     </visual>
+    <collision>
+      <origin xyz="0.497588819111708 0.333513492980419 -0.02" rpy="0 0 0" />
+      <geometry>
+        <box size="0.995177638223416 0.667026985960838 0.04"/>
+      </geometry>
+      <material name="wood">
+        <color rgba="0.713725490196078   0.607843137254902   0.298039215686275 1.0"/>
+      </material>
+    </collision>
     <inertial>
         <origin xyz="0 0 0" rpy="0 0 0" />
@@ -31,4 +40,13 @@
       </material>
     </visual>
+    <collision>
+      <origin xyz="0 0 -0.4" rpy="0 0 0" />
+      <geometry>
+        <box size="0.9 0.6 0.8"/>
+      </geometry>
+      <material name="blue">
+        <color rgba="0   0   0.7 1.0"/>
+      </material>
+    </collision>
     <inertial>
         <origin xyz="0 0 0" rpy="0 0 0" />
