Commit message: marco: fix description

File: hrc_simulator_descriptions/urdf/hrc_simulator.xacro (robot description, xacro)
@@ -71,5 +71,5 @@
 <link name="floor">
   <collision>
-    <origin  xyz="0.0 0.0 -0.5" rpy="0 0 0" />
+    <origin  xyz="0.0 0.0 -0.6" rpy="0 0 0" />
     <geometry>
       <box size="8 8 1.0"/>
@@ -97,5 +97,5 @@
 <link name="wall2">
   <collision>
-    <origin  xyz="0.0 -0.5 1.5" rpy="0 0 0" />
+    <origin  xyz="0.0 -0.5 1.25" rpy="0 0 0" />
     <geometry>
       <box size="8 1 1.5"/>
@@ -106,5 +106,5 @@
   <parent link = "world" />
   <child  link = "wall2" />
-<origin xyz="2 -1 0" rpy="0 0 0.0" />
+<origin xyz="2 -1.5 0" rpy="0 0 0.0" />
 </joint>
 <link name="wall3">

Commit message: samuele-devel

File: hrc_simulator_descriptions/urdf/hrc_simulator.xacro (robot description, xacro)
@@ -71,5 +71,5 @@
 <link name="floor">
   <collision>
-    <origin  xyz="0.0 0.0 -0.6" rpy="0 0 0" />
+    <origin  xyz="0.0 0.0 -1" rpy="0 0 0" />
     <geometry>
       <box size="8 8 1.0"/>

Commit message: Modified tabletop position

File: hrc_simulator_descriptions/urdf/hrc_simulator.xacro (robot description, xacro)
@@ -67,5 +67,5 @@
   <parent link = "world" />
   <child  link = "tabletop" />
-  <origin xyz="1.73 1.72 1.04" rpy="0 0 ${-0.5*pi}" />
+  <origin xyz="-0.3 2.8 1.04" rpy="0 0 ${-0.0*pi}" />
 </joint>
 <link name="floor">

Commit message: Simulations

File: hrc_simulator_descriptions/urdf/hrc_simulator.xacro (robot description, xacro)
@@ -24,5 +24,5 @@
   <parent link="world" />
   <child  link = "origin_human14dof" />
-  <origin xyz="1 1 0.0" rpy="0 0 ${-0.5*pi}" />
+  <origin xyz="1.5 1.2 0.0" rpy="0 0 ${-0.5*pi}" />
 </joint>
 <link name="tip">
@@ -57,15 +57,15 @@
   <parent link = "world" />
   <child  link = "shopdesk" />
-<origin xyz="1 -0.95 0.94" rpy="0.0 0.0 ${-0.0*pi}" />
+<origin xyz="2.1 -1.0 0.94" rpy="0.0 0.0 ${-0.0*pi}" />
 </joint>
 <joint name="elmo_linear_guide_fixed" type="fixed">
   <parent link = "world" />
   <child  link = "elmo_linear_guide_stator" />
-  <origin xyz="0.090 -0.32 0.95" rpy="0 0 0.005" />
+  <origin xyz="0.5 -0.32 0.95" rpy="0 0 0.005" />
 </joint>
 <joint name="tabletop_fixed" type="fixed">
   <parent link = "world" />
   <child  link = "tabletop" />
-  <origin xyz="-0.3 2.8 1.04" rpy="0 0 ${-0.0*pi}" />
+  <origin xyz="-0.9 2.4 1.04" rpy="0 0 ${0.5*pi}" />
 </joint>
 <link name="floor">
@@ -119,5 +119,5 @@
   <parent link = "world" />
   <child  link = "wall3" />
-<origin xyz="-0.3 2 0" rpy="0 0 0.0" />
+<origin xyz="-1.4 2 0" rpy="0 0 0.0" />
 </joint>
 <gazebo reference="world">

File: hrc_simulator_descriptions/urdf/shopdesk_dim.urdf.xacro (robot description, xacro)
@@ -6,5 +6,5 @@
       <origin xyz="0 0 -0.5" rpy="0 0 0" />
       <geometry>
-        <box size="2 0.8 1.0"/>
+        <box size="1 0.8 1.0"/>
       </geometry>
       <material name="sabbia">
@@ -23,5 +23,5 @@
       <origin xyz="0 0 -0.8" rpy="0 0 0" />
       <geometry>
-        <box size="2.04 0.84 1.6"/>
+        <box size="1.04 0.84 1.6"/>
       </geometry>
       <material name="sabbia">
