Commit message: left arm bent down: joint position changed

File: hrc_simulator_descriptions/urdf/human14dof/human_only_arms.urdf.xacro (robot description, xacro)
@@ -437,5 +437,5 @@
 	  <!--Chain from (12) to (15)-->
 	  <joint name="jLeftShoulder_rotx" type="revolute">
-          <origin xyz="0 ${Chest_box_y/2} ${Chest_box_z-UpperArm_radius}" rpy="0 0 0"/>
+          <origin xyz="0 ${Chest_box_y/2} ${Chest_box_z-UpperArm_radius}" rpy="-1.0472 0 0"/>
           <parent link="Chest"/>
           <child link="LeftUpperArm_f1"/>
@@ -476,5 +476,5 @@
         </joint>
       <joint name="jLeftElbow_roty" type="fixed">
-          <origin xyz="0     ${UpperArm_length}           0" rpy="0 0 0"/>
+          <origin xyz="0     ${UpperArm_length}           0" rpy="-0.4 0 0"/>
           <parent link="LeftUpperArm"/>
           <child link="LeftForeArm_f1"/>
